File: sensors/sensors.kicad_sch (KiCad schematic)
At the start: 6 parts, among them J1 Conn 1x3, U1 TCRT5000

Commit message: Submitted for reveiw
Parts:
- R1: value R -> 50R
- R2: value R -> 2k
Changed lines of the file:
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@@
 			)
 		)
-		(property "Value" "R"
+		(property "Value" "2k"
 			(at 138.43 92.7099 0)
 			(effects
@@
 			)
 		)
-		(property "Value" "R"
+		(property "Value" "50R"
 			(at 97.79 92.7099 0)
 			(effects
