File: other stuff/sensors/sensors.kicad_pcb (KiCad board)
At the start: 2 copper layers, 20 x 50 mm, 6 parts, among them J1 Conn_01x03_Pin, U1 TCRT5000

Commit message: Added files from 'Curtis', and updated 'sensors'
Parts:
- H1, H2: footprint MountingHole:MountingHole_4.3mm_M4 -> MountingHole:MountingHole_3.2mm_M3
- J1: value Conn_01x03_Pin -> Conn 1x3
- R1: value R -> 50R
- R2: value R -> 2k
- U1: footprint footprints:TCRT5000_VIS -> TCRT5000:OPTO_TCRT5000
- moved U1 4.04 mm to (160.2, 92.8)
Routing:
- net Vss: track 20.3 -> 18.5 mm
- net Vout: track 20.0 -> 18.3 mm
- net Net-(R2-Pad1): track 7.61 -> 5.92 mm
