File: other stuff/sensors/sensors.kicad_sch (KiCad schematic)
At the start: 6 parts, among them J1 Conn 1x3, U1 TCRT5000

Commit message: Added files from 'Curtis', and updated 'sensors'
Parts:
- H1, H2: footprint MountingHole:MountingHole_4.3mm_M4 -> MountingHole:MountingHole_3.2mm_M3
- U1: footprint footprints:TCRT5000_VIS -> TCRT5000:OPTO_TCRT5000
Changed lines of the file:
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@@
 			)
 		)
-		(property "Footprint" "MountingHole:MountingHole_4.3mm_M4"
+		(property "Footprint" "MountingHole:MountingHole_3.2mm_M3"
 			(at 50.8 44.45 0)
 			(effects
@@
 			)
 		)
-		(property "Footprint" "MountingHole:MountingHole_4.3mm_M4"
+		(property "Footprint" "MountingHole:MountingHole_3.2mm_M3"
 			(at 50.8 114.3 0)
 			(effects
@@
 			)
 		)
-		(property "Footprint" "footprints:TCRT5000_VIS"
+		(property "Footprint" "TCRT5000:OPTO_TCRT5000"
 			(at 95.25 80.01 0)
 			(effects
