File: pcb_draft_lfr/pcb_draft_lfr.kicad_sch (KiCad schematic)
At the start: 41 parts, among them J1 Conn_01x03_Pin, J2 Conn_01x02_Pin, J3 AVR-ISP-6, J4 Conn_01x03_Pin, J5 Conn_01x03_Pin, J6 Conn_01x03_Pin, J7 Conn_01x03_Pin, J8 Conn_01x02_Pin, J9 PINHD_1x4_Male, Q1 BSR802N, Q2 BSR802N, U1 TCRT5000, U2 MCP1700x-330xxTO, U4 ATMEGA328-PU, X1 HC49-SMD

Commit message: Readded files
Parts:
- C3, C4: value 33p -> 30p
Changed lines of the file:
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@@
 			)
 		)
-		(property "Value" "33p"
+		(property "Value" "30p"
 			(at 58.42 69.85 90)
 			(effects
@@
 		)
 		(property "Value" "10k"
-			(at 56.642 94.488 0)
+			(at 58.674 93.98 0)
 			(effects
 				(font
@@
 			)
 		)
-		(property "Value" "33p"
+		(property "Value" "30p"
 			(at 55.372 79.502 90)
 			(effects

Commit message: Submitted for reveiw
Parts:
- removed C9: 100n, Capacitor_SMD:C_1206_3216Metric_Pad1.33x1.80mm_HandSolder, symbol Device:C
- removed D1, D2: 1N4004, Diode_THT:D_DO-41_SOD81_P10.16mm_Horizontal, symbol Diode:1N4004
- removed J9: PINHD_1x4_Male, Connector_PinHeader_2.54mm:PinHeader_1x04_P2.54mm_Vertical, symbol PCM_SL_Pin_Headers:PINHD_1x4_Male
- removed L1, L2: 300u, symbol PCM_Generic-50:L,IEC
- removed R1, R9: 7, symbol PCM_Elektuur:R
- removed V1: 4.8, symbol Simulation_SPICE:VDC
- added BT1, BT2: 2462, 2462:BAT_2462, symbol 2462:2462
- added D3: LED_5mm (Green), LED_THT:LED_D5.0mm, symbol PCM_SL_Devices:LED_5mm
- added D4: LED_5mm (Red), LED_THT:LED_D5.0mm, symbol PCM_SL_Devices:LED_5mm
- added D5: LED_5mm (Blue), LED_THT:LED_D5.0mm, symbol PCM_SL_Devices:LED_5mm
- added D6, D7: SB130, Diode_THT:D_DO-41_SOD81_P10.16mm_Horizontal, symbol Diode:SB130
- added J10: Conn_01x04_Pin, Connector_PinHeader_2.54mm:PinHeader_1x04_P2.54mm_Vertical, symbol Connector:Conn_01x04_Pin
- added M1: Motor_DC, symbol Motor:Motor_DC
- added R10: 330, Resistor_THT:R_Axial_DIN0309_L9.0mm_D3.2mm_P12.70mm_Horizontal, symbol PCM_Elektuur:R
- added R11: 10k, Resistor_THT:R_Axial_DIN0309_L9.0mm_D3.2mm_P12.70mm_Horizontal, symbol PCM_Elektuur:R
- added R12: 120, Resistor_THT:R_Axial_DIN0309_L9.0mm_D3.2mm_P12.70mm_Horizontal, symbol PCM_Elektuur:R
- added R13: 140, Resistor_THT:R_Axial_DIN0309_L9.0mm_D3.2mm_P12.70mm_Horizontal, symbol PCM_Elektuur:R
- added R14: 20, Resistor_THT:R_Axial_DIN0309_L9.0mm_D3.2mm_P12.70mm_Horizontal, symbol PCM_Elektuur:R
- added S2: SPI Switch, digikey-footprints:Switch_Slide_JS202011SCQN, symbol dk_Slide-Switches:JS202011SCQN
- added S3: Button1 I/O, digikey-footprints:Switch_Tactile_THT_6x6mm_MJTP1230, symbol dk_Tactile-Switches:MJTP1230
- added TP1, TP2, TP3: TestPoint, TestPoint:TestPoint_2Pads_Pitch2.54mm_Drill0.8mm, symbol Connector:TestPoint
- J1, J4, J5, J6, J7: footprint (none) -> Connector_PinHeader_2.54mm:PinHeader_1x03_P2.54mm_Vertical
- J2, J8: footprint (none) -> Connector_PinHeader_2.54mm:PinHeader_1x02_P2.54mm_Vertical
- R2: value 3300 -> 3.9k
- R3: value 200 -> 100
- U1: footprint OptoDevice:Vishay_TCRT5000 -> TCRT5000:OPTO_TCRT5000
Connections:
- net Vbat+: now also BT2.P, D6.1 (K), D7.1 (K), M1.1 (+), TP1.1
- net Vcc: now also R10.2 (-), S2.1, S2.4; no longer C7.1, C8.1, U2.3 (VO)
- net Vgnd: now also BT1.N, D3.1, D4.1, D5.1, J10.1 (Pin_1), R11.1 (+), TP3.1
- net Vmotout: now also D7.2 (A), M1.2 (-)
- net Vre: now also J10.4 (Pin_4)
- net at U4.3 (PD1): now also J10.2 (Pin_2)
- net at U4.2 (PD0): now also J10.3 (Pin_3)
- net at U4.13 (PD7): now also R11.2 (-), S3.1, S3.2
- net at U4.14 (PB0): now also R12.1 (+)
- net at U4.15 (PB1): now also R13.1 (+)
- net Vmotout2: no longer names the net of J8.1 (Pin_1), Q2.3 (D)
- net Vmotout2: now also D6.2 (A)
- new net: D4.2, R13.2 (-)
- new net: C7.1, C8.1, S2.2, S2.5, TP2.1, U2.3 (VO)
- new net: R14.1 (+), S2.6
- new net: BT1.P, BT2.N
- new net: D5.2, R14.2 (-)
- new net: D3.2, R12.2 (-)
- new net: R10.1 (+), S3.3, S3.4
- no-connect marks 8 -> 7
Other:
- note added: "Both the motor and sensor will not be on this pcb"
- note added: "LED1-2 I/O"
- note added: "Label/naming convension incomplete"
- note added: "Motor 1 Connector"
- note added: "Motor 2 Connector"
- note added: "Reflector Sensor 1 Connector"
- note added: "Reset"
- note added: "Resistor values could be 200-260 ohms and 3300 ohms?"
- note added: "Sensor Connectors"
- note added: "Serial Port for Debugging"
- note added: "Should/Can we add ferrit beads?"
- note added: "Timer"
- note added: "Voltage Regulator"
- note removed: "Motor 1"
- note removed: "Motor 2"
- note removed: "Reflector Sensor 1"
- title: (none) -> LFR PCB Draft Schematic
- moved on the sheet: C11, J2, J3, J8, Q1, Q2, R2, R3, R6, R7, R8, U1

Commit message: Submitted for reveiw
Parts:
- removed BT1, BT2: 2462, 2462:BAT_2462, symbol 2462:2462
- removed M1: Motor_DC, symbol Motor:Motor_DC
- removed R2: 3.9k, Resistor_THT:R_Axial_DIN0309_L9.0mm_D3.2mm_P12.70mm_Horizontal, symbol PCM_Elektuur:R
- removed R3: 100, Resistor_SMD:R_0805_2012Metric_Pad1.20x1.40mm_HandSolder, symbol PCM_Elektuur:R
- removed U1: TCRT5000, TCRT5000:OPTO_TCRT5000, symbol TCRT5000:TCRT5000
- added H1, H2, H3, H4: MountingHole, MountingHole:MountingHole_3.2mm_M3, symbol Mechanical:MountingHole
- added J10: Conn_01x02_Pin, Connector_PinHeader_2.54mm:PinHeader_1x02_P2.54mm_Vertical, symbol Connector:Conn_01x02_Pin
- Q1, Q2: value BSR802N -> MOSFET N-Channel
- R1: renamed from R14; footprint Resistor_THT:R_Axial_DIN0309_L9.0mm_D3.2mm_P12.70mm_Horizontal -> Resistor_SMD:R_0805_2012Metric_Pad1.20x1.40mm_HandSolder
- R10: renamed from R6; footprint Resistor_THT:R_Axial_DIN0309_L9.0mm_D3.2mm_P12.70mm_Horizontal -> Resistor_SMD:R_0805_2012Metric_Pad1.20x1.40mm_HandSolder
- R3: renamed from R4; footprint Resistor_THT:R_Axial_DIN0309_L9.0mm_D3.2mm_P12.70mm_Horizontal -> Resistor_SMD:R_0805_2012Metric_Pad1.20x1.40mm_HandSolder
- R4: renamed from R10; footprint Resistor_THT:R_Axial_DIN0309_L9.0mm_D3.2mm_P12.70mm_Horizontal -> Resistor_SMD:R_0805_2012Metric_Pad1.20x1.40mm_HandSolder
- R6: renamed from R12; footprint Resistor_THT:R_Axial_DIN0309_L9.0mm_D3.2mm_P12.70mm_Horizontal -> Resistor_SMD:R_0805_2012Metric_Pad1.20x1.40mm_HandSolder
- R7: renamed from R13; footprint Resistor_THT:R_Axial_DIN0309_L9.0mm_D3.2mm_P12.70mm_Horizontal -> Resistor_SMD:R_0805_2012Metric_Pad1.20x1.40mm_HandSolder
- R8: footprint Resistor_THT:R_Axial_DIN0309_L9.0mm_D3.2mm_P12.70mm_Horizontal -> Resistor_SMD:R_0805_2012Metric_Pad1.20x1.40mm_HandSolder
- R9: renamed from R7; footprint Resistor_THT:R_Axial_DIN0309_L9.0mm_D3.2mm_P12.70mm_Horizontal -> Resistor_SMD:R_0805_2012Metric_Pad1.20x1.40mm_HandSolder
- S1: value MJTP1230 -> Reset Button
- S3: renamed from S2; value SPI Switch -> SPI On/Off Switch; footprint digikey-footprints:Switch_Slide_JS202011SCQN -> footprints:SWITCH_011CQN
- TP1, TP2, TP3: footprint TestPoint:TestPoint_2Pads_Pitch2.54mm_Drill0.8mm -> TestPoint:TestPoint_Pad_D2.0mm
- U1: renamed from U2; value MCP1700x-330xxTO -> Voltage Regulator
- X1: value HC49-SMD -> Crystal SMD
- renumbered C11 to C1, C4 to C10, C6 to C2, C7 to C3, C10 to C4, C8 to C5, C2 to C6, C5 to C7, C1 to C8, C3 to C9, D7 to D1, D6 to D2, D5 to D3, D3 to D4, D4 to D5, J4 to J2, J5 to J3, J6 to J4, J7 to J5, J2 to J6, J8 to J7, J10 to J8, J3 to J9, R5 to R2, R11 to R5, S3 to S2, U4 to U2
Connections:
- net Vbat+: now also TP2.1, J10.2 (Pin_2); no longer TP1.1
- net Button1: now reaches R5.2 (-), S2.1, S2.2, U2.13 (PD7)
- net TXD: now reaches J8.2 (Pin_2), U2.3 (PD1)
- net RXD: now reaches J8.3 (Pin_3), U2.2 (PD0)
- net LED2: now reaches R7.1 (+), U2.15 (PB1)
- net at C3.1, C5.1, S3.2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: now also TP3.1; no longer TP2.1
- net XTAL1: now reaches C9.2, U2.9 (PB6), X1.2
- net LED1: now reaches R6.1 (+), U2.14 (PB0)
- net XTAL2: now reaches C10.2, U2.10 (PB7), X1.1
- net Vgnd renamed GND
- net GND: now also TP1.1, J10.1 (Pin_1); no longer TP3.1
- net Vmotout: no longer names the net of D1.2 (A), J6.1 (Pin_1), Q1.3 (D)
Other:
- note added: "Button 1 I/O Circuit"
- note added: "LED 1 and 2 I/O Circuit"
- note added: "Microcontroller"
- note added: "Motor Driver Circuit"
- note added: "Mounting Holes (M3)"
- note added: "Reset Circuit"
- note added: "Serial Port Input (SPI)"
- note added: "Timer Circuit"
- note added: "Voltage Regulator Circuit"
- note removed: "Both the motor and sensor will not be on this pcb"
- note removed: "LED1-2 I/O"
- note removed: "Label/naming convension incomplete"
- note removed: "Motor 1 (Example)"
- note removed: "Reflector Sensor 1 (Example)"
- note removed: "Reflector Sensor 1 Connector"
- note removed: "Reset"
- note removed: "Resistor values could be 200-260 ohms and 3300 ohms?"
- note removed: "Serial Port Input"
- note removed: "Should/Can we add ferrit beads?"
- note removed: "Timer"
- note removed: "Voltage Regulator"
- moved on the sheet: C1, C10, C6, C7, C8, C9, D1, D2, D4, D5, J1, J2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

Commit message: Fixed the switch, and added more vias to ground for the mosfets.
Connections:
- net Vcc: now also S3.6; no longer S3.4
- net at R1.1 (+): now also S3.4; no longer S3.6
