File: pcb_draft_lfr/pcb_draft_lfr.kicad_sch (KiCad schematic)
At the start: 50 parts, among them J1 Conn_01x03_Pin, J10 Conn_01x02_Pin, J2 Conn_01x03_Pin, J3 Conn_01x03_Pin, J4 Conn_01x03_Pin, J5 Conn_01x03_Pin, J6 Conn_01x02_Pin, J7 Conn_01x02_Pin, J8 Conn_01x04_Pin, J9 AVR-ISP-6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

Commit message: handin
Parts:
- J1: value Conn_01x03_Pin -> Conn_Sens_1
- J10: value Conn_01x02_Pin -> Conn_Battery
- J2: value Conn_01x03_Pin -> Conn_Sens_2
- J3: value Conn_01x03_Pin -> Conn_Sens_3
- J4: value Conn_01x03_Pin -> Conn_Sens_4
- J5: value Conn_01x03_Pin -> Conn_Sens_5
- J6: value Conn_01x02_Pin -> Conn_Motor_1
- J7: value Conn_01x02_Pin -> Conn_Motor_2
- J8: value Conn_01x04_Pin -> Conn_Debug
- TP1: value TestPoint -> TestPoint_GND
- TP2: value TestPoint -> TestPoint_Vbattery
- TP3: value TestPoint -> TestPoint_Vcc
Other:
- note added: "Serial Port Interface (SPI)"
- note removed: "Serial Port Input (SPI)"
Changed lines of the file:
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@@
 		)
 	)
-	(text "Serial Port Input (SPI)"
+	(text "Serial Port Interface (SPI)"
 		(exclude_from_sim no)
 		(at 30.48 23.622 0)
@@
 	(wire
 		(pts
-			(xy 250.19 118.11) (xy 250.19 123.19)
-		)
-		(stroke
-			(width 0)
-			(type default)
-		)
-	)
-	(wire
-		(pts
 			(xy 100.33 181.61) (xy 100.33 185.42)
 		)
@@
 	(wire
 		(pts
+			(xy 250.19 118.11) (xy 250.19 123.19)
+		)
+		(stroke
+			(width 0)
+			(type default)
+		)
+	)
+	(wire
+		(pts
 			(xy 46.99 95.25) (xy 52.07 95.25)
 		)
@@
 			)
 		)
-		(property "Value" "Conn_01x02_Pin"
+		(property "Value" "Conn_Battery"
 			(at 218.44 126.3649 90)
 			(effects
@@
 			)
 		)
-		(property "Value" "Conn_01x04_Pin"
+		(property "Value" "Conn_Debug"
 			(at 152.908 94.488 0)
 			(effects
@@
 		(on_board yes)
 		(dnp no)
-		(fields_autoplaced yes)
 		(property "Reference" "J7"
 			(at 256.54 115.5699 0)
@@
 			)
 		)
-		(property "Value" "Conn_01x02_Pin"
+		(property "Value" "Conn_Motor_2"
 			(at 256.54 118.1099 0)
 			(effects
@@
 			)
 		)
-		(property "Value" "Conn_01x03_Pin"
+		(property "Value" "Conn_Sens_3"
 			(at 116.078 166.37 0)
 			(effects
@@
 			)
 		)
-		(property "Value" "Conn_01x03_Pin"
+		(property "Value" "Conn_Sens_1"
 			(at 80.518 169.164 0)
 			(effects
@@
 			)
 		)
-		(property "Value" "Conn_01x02_Pin"
+		(property "Value" "Conn_Motor_1"
 			(at 256.54 138.4299 0)
 			(effects
@@
 			)
 		)
-		(property "Value" "TestPoint"
+		(property "Value" "TestPoint_Vbattery"
 			(at 255.27 124.4599 90)
 			(effects
@@
 		(on_board yes)
 		(dnp no)
-		(fields_autoplaced yes)
 		(property "Reference" "TP3"
 			(at 212.09 25.9079 0)
@@
 			)
 		)
-		(property "Value" "TestPoint"
-			(at 212.09 28.4479 0)
+		(property "Value" "TestPoint_Vcc"
+			(at 212.09 27.686 0)
 			(effects
 				(font
@@
 			)
 		)
-		(property "Value" "TestPoint"
-			(at 195.326 124.714 90)
+		(property "Value" "TestPoint_GND"
+			(at 193.802 124.46 90)
 			(effects
 				(font
@@
 			)
 		)
-		(property "Value" "Conn_01x03_Pin"
+		(property "Value" "Conn_Sens_4"
 			(at 133.858 168.91 0)
 			(effects
@@
 			)
 		)
-		(property "Value" "Conn_01x03_Pin"
+		(property "Value" "Conn_Sens_5"
 			(at 151.638 168.91 0)
 			(effects
@@
 			)
 		)
-		(property "Value" "Conn_01x03_Pin"
+		(property "Value" "Conn_Sens_2"
 			(at 98.806 169.164 0)
 			(effects
