File: pcb_draft_lfr/pcb_draft_lfr.kicad_pcb (KiCad board)
At the start: 2 copper layers, 54.8 x 64.6 mm, 50 parts, among them J1 Conn_01x03_Pin, J10 Conn_01x02_Pin, J2 Conn_01x03_Pin, J3 Conn_01x03_Pin, J4 Conn_01x03_Pin, J5 Conn_01x03_Pin, J6 Conn_01x02_Pin, J7 Conn_01x02_Pin, J8 Conn_01x04_Pin, J9 AVR-ISP-6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

Commit message: REV3/4
Parts:
- moved C3 44.3 mm to (137.9, 131.0), turned to 90 degrees
- moved C5 39.4 mm to (133.6, 130.1), turned to 90 degrees
- moved C2 38.1 mm to (121.7, 130.7), turned to 90 degrees
- moved C4 37.3 mm to (126.3, 130.2), turned to 90 degrees
- moved H4 37.0 mm to (140.1, 114.6)
- moved U1 36.3 mm to (129.6, 129.0), turned to -90 degrees
- moved TP1 35.0 mm to (126.0, 137.4)
- moved D3 31.8 mm to (139.5, 123.9), turned to 180 degrees
- moved S3 26.6 mm to (125.0, 124.6), turned to 90 degrees
- moved R1 25.8 mm to (133.9, 123.3)
- moved TP2 25.5 mm to (129.5, 137.3)
- moved J7 22.4 mm to (129.5, 144.6)
- moved TP3 21.2 mm to (133.2, 137.3)
- moved J10 19.7 mm to (133.1, 144.6)
- moved Q1 18.9 mm to (113.0, 144.9)
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Routing:
- net GND: track 125.2 -> 19.2 mm, vias 12 -> 6
- net Vgate1: track 25.9 -> 44.9 mm
- net Net-(J9-SCK): track 30.8 -> 44.7 mm, vias 2 -> 0
- net Vcc: track 104.7 -> 91.4 mm, vias 2 -> 0
- net Vgate2: track 15.3 -> 27.4 mm
- net Net-(R1-+): track 4.95 -> 14.1 mm
- net Net-(J9-MOSI): track 46.8 -> 53.6 mm, vias 2 -> 0
- net Net-(U1-VO): track 40.2 -> 33.5 mm, vias 1 -> 0
- net Vmiso: track 8.64 -> 2.04 mm
- net Net-(D2-A): track 13.3 -> 19.2 mm
- net Vbat+: track 65.3 -> 60.6 mm
- net Net-(D1-A): track 17.5 -> 12.8 mm
- net Button1: track 38.1 -> 35.1 mm
- net TXD: track 15.2 -> 13.0 mm
- net RXD: track 15.2 -> 13.0 mm
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Other:
- board size 54.8 x 64.6 mm -> 42.7 x 75.7 mm

Commit message: REV3/4
Parts:
- moved R9 0.60 mm to (127.7, 110.4)
- moved J8 0.41 mm to (104.3, 92.2)
Routing:
- net Net-(J9-MOSI): track 53.6 -> 54.1 mm
- net Vsens1: track 16.9 -> 17.2 mm, vias 1 -> 2
- net Vsens2: track 15.2 -> 15.5 mm, vias 1 -> 2
- net Vsens4: track 14.1 -> 14.2 mm, vias 1 -> 2
- net Vsens5: vias 1 -> 2
- net Vsens3: vias 1 -> 2

Commit message: REV4
Routing:
- net Vgate1: track 44.9 -> 46.7 mm
Changed lines of the file:
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@@
 	(title_block
 		(title "PCB Design")
-		(rev "REV3")
+		(rev "REV4")
 		(comment 1 "Continued reveiw with fixes/changes made. + improvements")
+		(comment 2 "Do you want the MOSFET to ground to be bigger than 2mm?")
 	)
 	(layers
@@
 	)
 	(segment
-		(start 108.008 118.368)
-		(end 108.008 116.592)
-		(width 0.254)
-		(layer "F.Cu")
-		(net 24)
-	)
-	(segment
-		(start 108.008 116.592)
-		(end 108.688 115.912)
-		(width 0.254)
-		(layer "F.Cu")
-		(net 24)
-	)
-	(segment
 		(start 103.722 132.422)
-		(end 103.722 122.654)
+		(end 103.722 117.742)
 		(width 0.254)
 		(layer "F.Cu")
@@
 	)
 	(segment
-		(start 108.688 115.912)
-		(end 109.728 115.912)
+		(start 111.8 140.5)
+		(end 103.722 132.422)
 		(width 0.254)
 		(layer "F.Cu")
@@
 	)
 	(segment
-		(start 111.8 143.95)
-		(end 111.8 140.5)
+		(start 108.236 113.228)
+		(end 112.412 113.228)
 		(width 0.254)
 		(layer "F.Cu")
@@
 	)
 	(segment
-		(start 109.728 115.912)
-		(end 117.1 108.54)
+		(start 103.722 117.742)
+		(end 108.236 113.228)
 		(width 0.254)
 		(layer "F.Cu")
@@
 	)
 	(segment
-		(start 111.8 140.5)
-		(end 103.722 132.422)
+		(start 112.412 113.228)
+		(end 117.1 108.54)
 		(width 0.254)
 		(layer "F.Cu")
@@
 	)
 	(segment
-		(start 103.722 122.654)
-		(end 108.008 118.368)
+		(start 111.8 143.95)
+		(end 111.8 140.5)
 		(width 0.254)
 		(layer "F.Cu")

Commit message: handin
Parts:
- J1: value Conn_01x03_Pin -> Conn_Sens_1
- J10: value Conn_01x02_Pin -> Conn_Battery
- J2: value Conn_01x03_Pin -> Conn_Sens_2
- J3: value Conn_01x03_Pin -> Conn_Sens_3
- J4: value Conn_01x03_Pin -> Conn_Sens_4
- J5: value Conn_01x03_Pin -> Conn_Sens_5
- J6: value Conn_01x02_Pin -> Conn_Motor_1
- J7: value Conn_01x02_Pin -> Conn_Motor_2
- J8: value Conn_01x04_Pin -> Conn_Debug
- TP1: value TestPoint -> TestPoint_GND
- TP2: value TestPoint -> TestPoint_Vbattery
- TP3: value TestPoint -> TestPoint_Vcc
- moved H2 2.11 mm to (105.8, 143.9)
Other:
- board text added: "LFR Group 32"
